File: PCBS/SWITCHES/SWITCHES.kicad_sch (KiCad schematic)
At the start: 19 parts, among them J1 Conn_01x03_Pin, J2 Conn_01x02_Socket, J3 Conn_01x02_Socket, J6 Conn_01x02_Socket, J7 Conn_01x02_Socket, U1 CD4043BPWR

Commit message: Completed. SilkScreen changes necessary
Uses one SMD right pin header socket for the rotary switch
Parts:
- added J8: Conn_01x03_Socket, Connector_PinSocket_2.54mm:PinSocket_1x03_P2.54mm_Vertical, symbol DigitalLogicLibrary:Conn_01x03_Socket
- J2: footprint Connector_PinHeader_2.54mm:PinHeader_1x02_P2.54mm_Vertical -> Connector_PinSocket_2.54mm:PinSocket_1x02_P2.54mm_Vertical
- J6: footprint Connector_PinHeader_2.54mm:PinHeader_1x02_P2.54mm_Vertical -> Connector_PinSocket_2.54mm:PinSocket_1x02_P2.54mm_Vertical_SMD_Pin1Right
Connections:
- net DEBOUNCE1: now also J1.2 (Pin_2)
- net DEBOUNCE2: no longer J1.2 (Pin_2)
- net OUTPUT1: now also J8.1 (Pin_1), J8.2 (Pin_2), J8.3 (Pin_3)
Changed lines of the file:
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@@
   (junction (at 50.8 101.6) (diameter 0) (color 0 0 0 0)
   )
+  (junction (at 254 123.19) (diameter 0) (color 0 0 0 0)
+  )
   (junction (at 193.04 154.94) (diameter 0) (color 0 0 0 0)
   )
@@
   )
   (junction (at 248.92 156.21) (diameter 0) (color 0 0 0 0)
+  )
+  (junction (at 254 120.65) (diameter 0) (color 0 0 0 0)
   )
   (no_connect (at 157.48 49.53))
@@
     (stroke (width 0) (type default))
   )
+  (wire (pts (xy 241.3 120.65) (xy 254 120.65))
+    (stroke (width 0) (type default))
+  )
   (wire (pts (xy 86.36 101.6) (xy 90.17 101.6))
     (stroke (width 0) (type default))
@@
     (stroke (width 0) (type default))
   )
+  (wire (pts (xy 254 123.19) (xy 254 125.73))
+    (stroke (width 0) (type default))
+  )
   (wire (pts (xy 193.04 154.94) (xy 193.04 156.21))
     (stroke (width 0) (type default))
@@
   )
   (wire (pts (xy 134.62 52.07) (xy 130.81 52.07))
+    (stroke (width 0) (type default))
+  )
+  (wire (pts (xy 254 120.65) (xy 254 123.19))
     (stroke (width 0) (type default))
   )
@@
     (effects (font (size 1.27 1.27)) (justify left bottom))
   )
+  (label "DEBOUNCE1" (at 227.33 57.15 0) (fields_autoplaced)
+    (effects (font (size 1.27 1.27)) (justify left bottom))
+  )
   (label "DEBOUNCE3" (at 161.29 46.99 0) (fields_autoplaced)
     (effects (font (size 1.27 1.27)) (justify left bottom))
@@
     (effects (font (size 1.27 1.27)) (justify left bottom))
   )
-  (label "DEBOUNCE2" (at 227.33 57.15 0) (fields_autoplaced)
-    (effects (font (size 1.27 1.27)) (justify left bottom))
-  )
   (label "VCC_RES" (at 227.33 54.61 0) (fields_autoplaced)
     (effects (font (size 1.27 1.27)) (justify left bottom))
@@
   )
   (label "OUTPUT1" (at 69.85 151.13 90) (fields_autoplaced)
+    (effects (font (size 1.27 1.27)) (justify left bottom))
+  )
+  (label "OUTPUT1" (at 241.3 120.65 0) (fields_autoplaced)
     (effects (font (size 1.27 1.27)) (justify left bottom))
   )
@@
         (path "/ee51f292-e26d-4592-addf-9e4720b689f5"
           (reference "J7") (unit 1)
+        )
+      )
+    )
+  )
+  (symbol (lib_id "DigitalLogicLibrary:Conn_01x03_Socket") (at 259.08 123.19 0) (unit 1)
+    (in_bom yes) (on_board yes) (dnp no) (fields_autoplaced)
+    (property "Reference" "J8" (at 260.35 121.92 0)
+      (effects (font (size 1.27 1.27)) (justify left))
+    )
+    (property "Value" "Conn_01x03_Socket" (at 260.35 124.46 0)
+      (effects (font (size 1.27 1.27)) (justify left))
+    )
+    (property "Footprint" "Connector_PinSocket_2.54mm:PinSocket_1x03_P2.54mm_Vertical" (at 259.08 123.19 0)
+      (effects (font (size 1.27 1.27)) hide)
+    )
+    (property "Datasheet" "~" (at 259.08 123.19 0)
+      (effects (font (size 1.27 1.27)) hide)
+    )
+    (pin "1")
+    (pin "2")
+    (pin "3")
+    (instances
+      (project "SWITCHES"
+        (path "/ee51f292-e26d-4592-addf-9e4720b689f5"
+          (reference "J8") (unit 1)
         )
       )
@@
       (effects (font (size 1.27 1.27)) (justify left))
     )
-    (property "Footprint" "Connector_PinHeader_2.54mm:PinHeader_1x02_P2.54mm_Vertical" (at 254 137.16 0)
+    (property "Footprint" "Connector_PinSocket_2.54mm:PinSocket_1x02_P2.54mm_Vertical_SMD_Pin1Right" (at 254 137.16 0)
       (effects (font (size 1.27 1.27)) hide)
     )
@@
       (effects (font (size 1.27 1.27)) (justify left))
     )
-    (property "Footprint" "Connector_PinHeader_2.54mm:PinHeader_1x02_P2.54mm_Vertical" (at 198.12 138.43 0)
-      (effects (font (size 1.27 1.27)) hide)
-    )
+    (property "Footprint" "Connector_PinSocket_2.54mm:PinSocket_1x02_P2.54mm_Vertical" (at 198.12 138.43 0)
+      (effects (font (size 1.27 1.27)) hide)
+    )

Commit message: Finished input PCB and fixed mux and not
Parts:
- added S2: 1571527-2, DigitalLogicFootprints:SW_1571527-2, symbol DigitalLogicLibrary:1571527-2
Connections:
- net DEBOUNCE1: now also S2.4
- net GND: now also S2.1
- net OUTPUT0: now also S2.2
- net VCC_RES: now also S2.3
Other:
- note added: "Push Button"
Changed lines of the file:
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@@
+    (stroke (width 0) (type default))
+  )
+  (wire (pts (xy 142.24 88.9) (xy 144.78 88.9))
     (stroke (width 0) (type default))
   )
@@
     (stroke (width 0) (type default))
   )
+  (wire (pts (xy 160.02 88.9) (xy 162.56 88.9))
+    (stroke (width 0) (type default))
+  )
   (wire (pts (xy 224.79 57.15) (xy 227.33 57.15))
     (stroke (width 0) (type default))
@@
     (stroke (width 0) (type default))
   )
+  (wire (pts (xy 142.24 93.98) (xy 144.78 93.98))
+    (stroke (width 0) (type default))
+  )
   (wire (pts (xy 248.92 154.94) (xy 248.92 156.21))
     (stroke (width 0) (type default))
@@
   )
   (wire (pts (xy 41.91 99.06) (xy 41.91 100.33))
+    (stroke (width 0) (type default))
+  )
+  (wire (pts (xy 160.02 93.98) (xy 163.83 93.98))
     (stroke (width 0) (type default))
   )
@@
     (effects (font (size 5 5)) (justify left bottom))
   )
+  (text "Push Button" (at 137.16 104.14 0)
+    (effects (font (size 2 2)) (justify left bottom))
+  )
   (text "Rotary Switch" (at 137.16 68.58 0)
     (effects (font (size 2 2)) (justify left bottom))
@@
     (effects (font (size 1.27 1.27)) (justify left bottom))
   )
+  (label "GND" (at 162.56 88.9 0) (fields_autoplaced)
+    (effects (font (size 1.27 1.27)) (justify left bottom))
+  )
   (label "OUTPUT3" (at 95.25 151.13 90) (fields_autoplaced)
     (effects (font (size 1.27 1.27)) (justify left bottom))
@@
     (effects (font (size 1.27 1.27)) (justify left bottom))
   )
+  (label "DEBOUNCE1" (at 142.24 93.98 180) (fields_autoplaced)
+    (effects (font (size 1.27 1.27)) (justify right bottom))
+  )
   (label "DEBOUNCE0" (at 38.1 109.22 0) (fields_autoplaced)
     (effects (font (size 1.27 1.27)) (justify left bottom))
@@
     (effects (font (size 1.27 1.27)) (justify left bottom))
   )
+  (label "VCC_RES" (at 142.24 88.9 180) (fields_autoplaced)
+    (effects (font (size 1.27 1.27)) (justify right bottom))
+  )
   (label "OUTPUT2" (at 82.55 151.13 90) (fields_autoplaced)
     (effects (font (size 1.27 1.27)) (justify left bottom))
@@
   )
   (label "DEBOUNCE1" (at 161.29 52.07 0) (fields_autoplaced)
+    (effects (font (size 1.27 1.27)) (justify left bottom))
+  )
+  (label "OUTPUT0" (at 163.83 93.98 0) (fields_autoplaced)
     (effects (font (size 1.27 1.27)) (justify left bottom))
   )
@@
         )
       )
+    )
+  )
+  (symbol (lib_id "DigitalLogicLibrary:1571527-2") (at 152.4 88.9 180) (unit 1)
+    (in_bom yes) (on_board yes) (dnp no) (fields_autoplaced)
+    (property "Reference" "S2" (at 152.4 76.2 0)
+      (effects (font (size 1.27 1.27)))
+    )
+    (property "Value" "1571527-2" (at 152.4 78.74 0)
+      (effects (font (size 1.27 1.27)))
+    )
+    (property "Footprint" "DigitalLogicFootprints:SW_1571527-2" (at 151.13 81.28 0)
+      (effects (font (size 1.27 1.27)) (justify bottom) hide)
+    )
+    (property "Datasheet" "" (at 152.4 88.9 0)
+      (effects (font (size 1.27 1.27)) hide)
+    )
+    (property "Comment" "1571527-2" (at 151.13 81.28 0)
+      (effects (font (size 1.27 1.27)) (justify bottom) hide)
+    )
+    (property "DigiKey_Part_Number" "" (at 152.4 88.9 0)
+      (effects (font (size 1.27 1.27)) (justify bottom) hide)
+    )
+    (property "MF" "TE Connectivity / AMP" (at 151.13 81.28 0)
+      (effects (font (size 1.27 1.27)) (justify bottom) hide)
+    )
+    (property "MAXIMUM_PACKAGE_HEIGHT" "5.25mm" (at 151.13 81.28 0)
+      (effects (font (size 1.27 1.27)) (justify bottom) hide)
+    )
+    (property "Package" "None" (at 151.13 81.28 0)
+      (effects (font (size 1.27 1.27)) (justify bottom) hide)
+    )
+    (property "Check_prices" "https://www.snapeda.com/parts/1571527-2/TE+Connectivity+%252F+AMP/view-part/?ref=eda" (at 152.4 83.82 0)
+      (effects (font (size 1.27 1.27)) (justify bottom) hide)
+    )
+    (property "STANDARD" "Manufacturer Recommendations" (at 151.13 81.28 0)
+      (effects (font (size 1.27 1.27)) (justify bottom) hide)
+    )
+    (property "PARTREV" "V" (at 151.13 81.28 0)
+      (effects (font (size 1.27 1.27)) (justify bottom) hide)
+    )
+    (property "SnapEDA_Link" "https://www.snapeda.com/parts/1571527-2/TE+Connectivity+%252F+AMP/view-part/?ref=snap" (at 151.13 81.28 0)
+      (effects (font (size 1.27 1.27)) (justify bottom) hide)
+    )
+    (property "MP" "1571527-2" (at 151.13 81.28 0)
+      (effects (font (size 1.27 1.27)) (justify bottom) hide)
+    )
+    (property "Purchase-URL" "https://www.snapeda.com/api/url_track_click_mouser/?unipart_id=491702&manufacturer=TE Connectivity / AMP&part_name=1571527-2&search_term=1571527-2" (at 151.13 81.28 0)
+      (effects (font (size 1.27 1.27)) (justify bottom) hide)
+    )
+    (property "EU_RoHS_Compliance" "Compliant" (at 151.13 81.28 0)
+      (effects (font (size 1.27 1.27)) (justify bottom) hide)
+    )
+    (property "Description" "\nSwitch Tactile OFF (ON) SPST Round Button Gull Wing 0.05A 24VDC 0.98N SMD T/R\n" (at 151.13 81.28 0)
+      (effects (font (size 1.27 1.27)) (justify bottom) hide)
+    )
+    (property "MANUFACTURER" "TE" (at 151.13 81.28 0)
+      (effects (font (size 1.27 1.27)) (justify bottom) hide)
+    )
+    (pin "1")
+    (pin "3")
+    (pin "4")
+    (pin "2")
+    (instances
+      (project "SWITCHES"
+        (path "/ee51f292-e26d-4592-addf-9e4720b689f5"
+          (reference "S2") (unit 1)
+        )
+      )
