File: PCBS/GATE/GATE.kicad_sch (KiCad schematic)
At the start: 13 parts, among them J1 Conn_01x01_Socket, J2 Conn_01x01_Socket, J3 Conn_01x03_Socket, U1 SN74LVC1G32DBVR

Commit message: Gate Rev 2 and Board Updates
Parts:
- added J6: Conn_01x01_Socket, Connector_PinSocket_2.54mm:PinSocket_1x01_P2.54mm_Vertical, symbol DigitalLogicLibrary:Conn_01x01_Socket
- added LED4: LTST-S220GKT, LED_LTST-S220GKT_LTO, symbol DigitalLogicLibrary:LTST-S220GKT
Connections:
- net NOT: now reaches J2.1 (Pin_1), LED2.2, U1.2 (B)
- net NOT: now also J6.1 (Pin_1), LED4.2
- net NOTRES: now reaches LED2.1, R2.1
- net NOTRES: now also LED4.1
Changed lines of the file:
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@@
 (kicad_sch (version 20230121) (generator eeschema)
   (paper "A4")
+  (junction (at 115.57 116.84) (diameter 0) (color 0 0 0 0)
+  )
   (junction (at 148.59 101.6) (diameter 0) (color 0 0 0 0)
   )
+  (junction (at 110.49 104.14) (diameter 0) (color 0 0 0 0)
+  )
   (junction (at 101.6 99.06) (diameter 0) (color 0 0 0 0)
   )
+  (junction (at 57.15 137.16) (diameter 0) (color 0 0 0 0)
+  )
   (junction (at 152.4 101.6) (diameter 0) (color 0 0 0 0)
   )
@@
     (stroke (width 0) (type default))
   )
+  (wire (pts (xy 57.15 152.4) (xy 57.15 147.32))
+    (stroke (width 0) (type default))
+  )
+  (wire (pts (xy 110.49 104.14) (xy 115.57 104.14))
+    (stroke (width 0) (type default))
+  )
   (wire (pts (xy 148.59 115.57) (xy 148.59 116.84))
     (stroke (width 0) (type default))
@@
     (stroke (width 0) (type default))
   )
+  (wire (pts (xy 101.6 116.84) (xy 101.6 115.57))
+    (stroke (width 0) (type default))
+  )
   (wire (pts (xy 130.81 87.63) (xy 130.81 88.9))
     (stroke (width 0) (type default))
@@
     (stroke (width 0) (type default))
   )
-  (wire (pts (xy 95.25 104.14) (xy 115.57 104.14))
+  (wire (pts (xy 95.25 104.14) (xy 110.49 104.14))
     (stroke (width 0) (type default))
   )
@@
     (stroke (width 0) (type default))
   )
+  (wire (pts (xy 48.26 137.16) (xy 57.15 137.16))
+    (stroke (width 0) (type default))
+  )
   (wire (pts (xy 130.81 114.3) (xy 130.81 116.84))
     (stroke (width 0) (type default))
   )
+  (wire (pts (xy 60.96 137.16) (xy 57.15 137.16))
+    (stroke (width 0) (type default))
+  )
   (wire (pts (xy 114.3 64.77) (xy 116.84 64.77))
     (stroke (width 0) (type default))
@@
     (stroke (width 0) (type default))
   )
+  (wire (pts (xy 60.96 134.62) (xy 60.96 137.16))
+    (stroke (width 0) (type default))
+  )
   (wire (pts (xy 96.52 64.77) (xy 99.06 64.77))
     (stroke (width 0) (type default))
@@
     (stroke (width 0) (type default))
   )
-  (wire (pts (xy 101.6 115.57) (xy 101.6 116.84))
+  (wire (pts (xy 113.03 116.84) (xy 115.57 116.84))
+    (stroke (width 0) (type default))
+  )
+  (wire (pts (xy 110.49 92.71) (xy 110.49 104.14))
+    (stroke (width 0) (type default))
+  )
+  (wire (pts (xy 48.26 152.4) (xy 57.15 152.4))
     (stroke (width 0) (type default))
   )
@@
     (stroke (width 0) (type default))
   )
+  (global_label "NOT" (shape input) (at 110.49 92.71 90) (fields_autoplaced)
+    (effects (font (size 1.27 1.27)) (justify left))
+    (property "Intersheetrefs" "${INTERSHEET_REFS}" (at 110.49 86.1756 90)
+      (effects (font (size 1.27 1.27)) (justify left) hide)
+    )
+  )
+  (global_label "NOTRES" (shape input) (at 48.26 152.4 180) (fields_autoplaced)
+    (effects (font (size 1.27 1.27)) (justify right))
+    (property "Intersheetrefs" "${INTERSHEET_REFS}" (at 38.0971 152.4 0)
+      (effects (font (size 1.27 1.27)) (justify right) hide)
+    )
+  )
+  (global_label "NOT" (shape input) (at 60.96 134.62 90) (fields_autoplaced)
+    (effects (font (size 1.27 1.27)) (justify left))
+    (property "Intersheetrefs" "${INTERSHEET_REFS}" (at 60.96 128.0856 90)
+      (effects (font (size 1.27 1.27)) (justify left) hide)
+    )
+  )
+  (global_label "NOTRES" (shape input) (at 113.03 116.84 180) (fields_autoplaced)
+    (effects (font (size 1.27 1.27)) (justify right))
+    (property "Intersheetrefs" "${INTERSHEET_REFS}" (at 102.8671 116.84 0)
+      (effects (font (size 1.27 1.27)) (justify right) hide)
+    )
+  )
   (symbol (lib_id "power:GND") (at 130.81 116.84 0) (unit 1)
     (in_bom yes) (on_board yes) (dnp no) (fields_autoplaced)
@@
     (pin "1")
     (instances
-      (project "ANDGATE"
+      (project "GATE"
         (path "/ee51f292-e26d-4592-addf-9e4720b689f5"
           (reference "#PWR04") (unit 1)
@@
     (pin "2")
     (instances
-      (project "ANDGATE"
+      (project "GATE"
         (path "/ee51f292-e26d-4592-addf-9e4720b689f5"
           (reference "LED3") (unit 1)
@@
     (pin "1")
     (instances
-      (project "ANDGATE"
+      (project "GATE"
         (path "/ee51f292-e26d-4592-addf-9e4720b689f5"
           (reference "#PWR05") (unit 1)
@@
     (pin "3")
     (instances
-      (project "ANDGATE"
+      (project "GATE"
         (path "/ee51f292-e26d-4592-addf-9e4720b689f5"
           (reference "J3") (unit 1)
@@
       (effects (font (size 1.27 1.27) italic) hide)
     )
-    (pin "2")
+    (pin "1")
+    (pin "2")
+    (pin "3")
     (pin "4")
     (pin "5")
-    (pin "1")
-    (pin "3")
-    (instances
-      (project "ANDGATE"
+    (instances
+      (project "GATE"
         (path "/ee51f292-e26d-4592-addf-9e4720b689f5"
           (reference "U1") (unit 1)
@@
     (pin "1")
     (instances
-      (project "ANDGATE"
+      (project "GATE"
         (path "/ee51f292-e26d-4592-addf-9e4720b689f5"
           (reference "J2") (unit 1)
@@
     (pin "2")
     (instances
-      (project "ANDGATE"
+      (project "GATE"
         (path "/ee51f292-e26d-4592-addf-9e4720b689f5"
           (reference "LED2") (unit 1)
@@
     (pin "1")
     (instances
-      (project "ANDGATE"
+      (project "GATE"
         (path "/ee51f292-e26d-4592-addf-9e4720b689f5"
           (reference "#PWR01") (unit 1)
@@
     (pin "1")
     (instances
-      (project "ANDGATE"
+      (project "GATE"
         (path "/ee51f292-e26d-4592-addf-9e4720b689f5"
           (reference "#PWR07") (unit 1)
@@
     (pin "1")
     (instances
-      (project "ANDGATE"
+      (project "GATE"
         (path "/ee51f292-e26d-4592-addf-9e4720b689f5"
           (reference "J5") (unit 1)
@@
     (pin "1")
     (instances
-      (project "ANDGATE"
+      (project "GATE"
         (path "/ee51f292-e26d-4592-addf-9e4720b689f5"
           (reference "#PWR02") (unit 1)
@@
     (pin "2")
     (instances
-      (project "ANDGATE"
+      (project "GATE"
         (path "/ee51f292-e26d-4592-addf-9e4720b689f5"
           (reference "LED1") (unit 1)
@@
     )
   )
+  (symbol (lib_id "DigitalLogicLibrary:Conn_01x01_Socket") (at 43.18 137.16 180) (unit 1)
+    (in_bom yes) (on_board yes) (dnp no) (fields_autoplaced)
+    (property "Reference" "J6" (at 43.815 132.08 0)
+      (effects (font (size 1.27 1.27)))
+    )
+    (property "Value" "Conn_01x01_Socket" (at 43.815 134.62 0)
+      (effects (font (size 1.27 1.27)))
+    )
+    (property "Footprint" "Connector_PinSocket_2.54mm:PinSocket_1x01_P2.54mm_Vertical" (at 43.18 137.16 0)
+      (effects (font (size 1.27 1.27)) hide)
+    )
+    (property "Datasheet" "~" (at 43.18 137.16 0)
+      (effects (font (size 1.27 1.27)) hide)
+    )
+    (pin "1")
+    (instances
+      (project "GATE"
+        (path "/ee51f292-e26d-4592-addf-9e4720b689f5"
+          (reference "J6") (unit 1)
+        )
+      )
+    )
+  )
   (symbol (lib_id "Device:R") (at 101.6 120.65 0) (unit 1)
     (in_bom yes) (on_board yes) (dnp no) (fields_autoplaced)
@@
     (pin "2")
     (instances
-      (project "ANDGATE"
+      (project "GATE"
         (path "/ee51f292-e26d-4592-addf-9e4720b689f5"
           (reference "R1") (unit 1)
@@
     (pin "1")
     (instances
-      (project "ANDGATE"
+      (project "GATE"
         (path "/ee51f292-e26d-4592-addf-9e4720b689f5"
           (reference "#PWR06") (unit 1)
@@
     (pin "1")
     (instances
-      (project "ANDGATE"
+      (project "GATE"
         (path "/ee51f292-e26d-4592-addf-9e4720b689f5"
           (reference "J1") (unit 1)
@@
     (pin "1")
     (instances
-      (project "ANDGATE"
+      (project "GATE"
         (path "/ee51f292-e26d-4592-addf-9e4720b689f5"
           (reference "#PWR03") (unit 1)
@@
       (effects (font (size 1.27 1.27)) (justify bottom) hide)
     )
+    (pin "1")
+    (pin "2")
     (pin "3")
-    (pin "2")
-    (pin "1")
     (pin "4")
     (instances
-      (project "ANDGATE"
+      (project "GATE"
         (path "/ee51f292-e26d-4592-addf-9e4720b689f5"
           (reference "D1") (unit 1)
@@
     )
   )
+  (symbol (lib_id "DigitalLogicLibrary:LTST-S220GKT") (at 57.15 137.16 270) (unit 1)
+    (in_bom yes) (on_board yes) (dnp no) (fields_autoplaced)
+    (property "Reference" "LED4" (at 63.5 142.24 90)
+      (effects (font (size 1.524 1.524)) (justify left))
+    )
+    (property "Value" "LTST-S220GKT" (at 63.5 144.78 90)
+      (effects (font (size 1.524 1.524)) (justify left))
+    )
+    (property "Footprint" "LED_LTST-S220GKT_LTO" (at 57.15 137.16 0)
+      (effects (font (size 1.27 1.27) italic) hide)
+    )
+    (property "Datasheet" "LTST-S220GKT" (at 57.15 137.16 0)
+      (effects (font (size 1.27 1.27) italic) hide)
+    )
+    (pin "1")
+    (pin "2")
+    (instances
+      (project "GATE"
+        (path "/ee51f292-e26d-4592-addf-9e4720b689f5"
+          (reference "LED4") (unit 1)
+        )
+      )
+    )
+  )
   (symbol (lib_id "Device:R") (at 115.57 120.65 0) (unit 1)
     (in_bom yes) (on_board yes) (dnp no) (fields_autoplaced)
@@
     (pin "2")
     (instances
-      (project "ANDGATE"
+      (project "GATE"
         (path "/ee51f292-e26d-4592-addf-9e4720b689f5"
           (reference "R2") (unit 1)
@@
     (pin "1")
     (instances
-      (project "ANDGATE"
+      (project "GATE"
         (path "/ee51f292-e26d-4592-addf-9e4720b689f5"
           (reference "J4") (unit 1)
@@
     (pin "2")
     (instances
-      (project "ANDGATE"
+      (project "GATE"
         (path "/ee51f292-e26d-4592-addf-9e4720b689f5"
           (reference "R3") (unit 1)
