File: PCBS/BOARD/BOARD.kicad_pcb (KiCad board)
At the start: 2 copper layers, 96 x 96 mm, 36 parts

Commit message: Gate Rev 2 and Board Updates
Parts:
- added S1: 1571527-2, DigitalLogicFootprints:SW_1571527-2, F.Cu at (111.8, 71.1)
- added S2: 1571527-2, DigitalLogicFootprints:SW_1571527-2, F.Cu at (111.8, 55.9)
- added U1: ATmega88PB-A, Package_QFP:TQFP-32_7x7mm_P0.8mm, F.Cu at (96.5, 55.9)

Commit message: Rev1 board/mux/switches/output
Parts:
- added D1: LTD-4708G, DigitalLogicFootprints:LED_LTD-4708G, F.Cu at (86.4, 48.0)
- added D2: 1N47xxA, Diode_THT:D_DO-41_SOD81_P10.16mm_Horizontal, B.Cu at (147.3, 71.1)
- added D3: 1N47xxA, Diode_THT:D_DO-41_SOD81_P10.16mm_Horizontal, B.Cu at (145.5, 58.4)
- added D4: 1N47xxA, Diode_THT:D_DO-41_SOD81_P10.16mm_Horizontal, F.Cu at (142.0, 58.4)
- added D5: 1N47xxA, Diode_THT:D_DO-41_SOD81_P10.16mm_Horizontal, B.Cu at (142.2, 71.1)
- added G***: LOGO, DigitalLogicFootprints:HBBLogo, B.Cu at (160.0, 129.5)
- added J37: Conn_01x03_Socket, DigitalLogicFootprints:PinHeader_1x03_P2.54mm_Vertical, F.Cu at (98.0, 48.0)
- added J38: USB_B_Micro, Connector_USB:USB_Micro-B_Amphenol_10118194_Horizontal, B.Cu at (143.2, 42.7)
- added J39: Conn_01x03_Socket, DigitalLogicFootprints:PinHeader_1x03_P2.54mm_Vertical, F.Cu at (98.0, 64.0)
- added J40: Conn_01x03_Socket, DigitalLogicFootprints:PinHeader_1x03_P2.54mm_Vertical, F.Cu at (98.0, 80.0)
- added J41: Conn_01x03_Socket, DigitalLogicFootprints:PinHeader_1x03_P2.54mm_Vertical, F.Cu at (98.0, 96.0)
- added J42: Conn_01x03_Socket, DigitalLogicFootprints:PinHeader_1x03_P2.54mm_Vertical, F.Cu at (98.0, 112.0)
- added J43: Conn_01x03_Socket, DigitalLogicFootprints:PinHeader_1x03_P2.54mm_Vertical, F.Cu at (98.0, 128.0)
- added J44: Conn_01x02_Pin, DigitalLogicFootprints:PinHeader_1x02_P2.54mm_Horizontal, F.Cu at (173.5, 88.0)
- added J45: Conn_01x02_Pin, DigitalLogicFootprints:PinHeader_1x02_P2.54mm_Horizontal, B.Cu at (127.0, 133.5)
- added J46: Conn_01x01_Socket, Connector_PinSocket_2.54mm:PinSocket_1x01_P2.54mm_Vertical, F.Cu at (175.0, 48.0)
- added J47: Conn_01x04_Socket, DigitalLogicFootprints:PinHeader_1x04_P2.54mm_Horizontal, B.Cu at (82.5, 72.0)
- added J48: Conn_01x04_Socket, DigitalLogicFootprints:PinHeader_1x04_P2.54mm_Horizontal, F.Cu at (173.5, 120.0)
- added J49: Conn_01x04_Socket, DigitalLogicFootprints:PinHeader_1x04_P2.54mm_Horizontal, F.Cu at (173.5, 72.0)
- added J50: Conn_01x04_Socket, DigitalLogicFootprints:PinHeader_1x04_P2.54mm_Horizontal, B.Cu at (82.5, 120.0)
- added J51: Conn_01x02_Pin, DigitalLogicFootprints:PinHeader_1x02_P2.54mm_Horizontal, F.Cu at (128.0, 42.5)
- added J52: Conn_01x01_Socket, Connector_PinSocket_2.54mm:PinSocket_1x01_P2.54mm_Vertical, F.Cu at (175.0, 64.0)
- added J53: Conn_01x01_Socket, Connector_PinSocket_2.54mm:PinSocket_1x01_P2.54mm_Vertical, F.Cu at (175.0, 80.0)
- added J54: Conn_01x01_Socket, Connector_PinSocket_2.54mm:PinSocket_1x01_P2.54mm_Vertical, F.Cu at (175.0, 96.0)
- added J55: Conn_01x01_Socket, Connector_PinSocket_2.54mm:PinSocket_1x01_P2.54mm_Vertical, F.Cu at (175.0, 112.0)
- added J56: Conn_01x04_Socket, DigitalLogicFootprints:PinHeader_1x04_P2.54mm_Horizontal, B.Cu at (112.0, 133.5)
- added J57: Conn_01x01_Socket, Connector_PinSocket_2.54mm:PinSocket_1x01_P2.54mm_Vertical, F.Cu at (175.0, 128.0)
- added J58: Conn_01x02_Pin, DigitalLogicFootprints:PinHeader_1x02_P2.54mm_Horizontal, B.Cu at (82.5, 88.0)
- added J59: Conn_01x04_Socket, DigitalLogicFootprints:PinHeader_1x04_P2.54mm_Horizontal, F.Cu at (112.0, 42.5)
- added J60: USB_B, Connector_USB:USB_B_OST_USB-B1HSxx_Horizontal, B.Cu at (158.7, 59.9)
- added J61: Conn_02x03_Counter_Clockwise, Connector_PinSocket_2.54mm:PinSocket_2x03_P2.54mm_Vertical, F.Cu at (94.0, 121.9)
- added LED1: LTST-S220GKT, DigitalLogicFootprints:LED_LTST-S220GKT_LTO, F.Cu at (98.0, 43.0)
- added LED10: LTST-S220GKT, DigitalLogicFootprints:LED_LTST-S220GKT_LTO, F.Cu at (173.0, 64.0)
- added LED11: LTST-S220GKT, DigitalLogicFootprints:LED_LTST-S220GKT_LTO, F.Cu at (173.0, 80.0)
- added LED12: LTST-S220GKT, DigitalLogicFootprints:LED_LTST-S220GKT_LTO, F.Cu at (173.0, 96.0)
- added LED13: LTST-S220GKT, DigitalLogicFootprints:LED_LTST-S220GKT_LTO, F.Cu at (173.0, 112.0)
- added LED14: LTST-S220GKT, DigitalLogicFootprints:LED_LTST-S220GKT_LTO, F.Cu at (173.0, 128.0)
- added LED2: LTST-S220GKT, DigitalLogicFootprints:LED_LTST-S220GKT_LTO, F.Cu at (98.0, 59.0)
- added LED3: LTST-S220GKT, DigitalLogicFootprints:LED_LTST-S220GKT_LTO, F.Cu at (98.0, 75.0)
- added LED4: LTST-S220GKT, DigitalLogicFootprints:LED_LTST-S220GKT_LTO, F.Cu at (98.0, 91.0)
- added LED5: LTST-S220GKT, DigitalLogicFootprints:LED_LTST-S220GKT_LTO, F.Cu at (94.0, 111.8)
- added LED6: LTST-S220GKT, DigitalLogicFootprints:LED_LTST-S220GKT_LTO, F.Cu at (98.0, 121.9)
- added LED9: LTST-S220GKT, DigitalLogicFootprints:LED_LTST-S220GKT_LTO, F.Cu at (173.0, 48.0)
- added Q1: NMOS, DigitalLogicFootprints:TO254P1041X444X1930-3, F.Cu at (88.9, 57.5)
- added R1: 510, Resistor_SMD:R_0805_2012Metric_Pad1.20x1.40mm_HandSolder, B.Cu at (127.0, 63.5)
- added R12: 510, Resistor_SMD:R_0805_2012Metric_Pad1.20x1.40mm_HandSolder, F.Cu at (172.7, 53.3)
- added R13: 510, Resistor_SMD:R_0805_2012Metric_Pad1.20x1.40mm_HandSolder, F.Cu at (172.0, 58.4)
- added R14: 510, Resistor_SMD:R_0805_2012Metric_Pad1.20x1.40mm_HandSolder, F.Cu at (172.7, 83.8)
- added R15: 510, Resistor_SMD:R_0805_2012Metric_Pad1.20x1.40mm_HandSolder, F.Cu at (173.5, 102.0)
- added R16: 510, Resistor_SMD:R_0805_2012Metric_Pad1.20x1.40mm_HandSolder, F.Cu at (167.6, 119.4)
- added R17: 510, Resistor_SMD:R_0805_2012Metric_Pad1.20x1.40mm_HandSolder, F.Cu at (172.7, 134.6)
- added R2: 510, Resistor_SMD:R_0805_2012Metric_Pad1.20x1.40mm_HandSolder, B.Cu at (134.6, 71.1)
- added R20: 510, Resistor_SMD:R_0805_2012Metric_Pad1.20x1.40mm_HandSolder, F.Cu at (94.0, 81.3)
- added R21: 510, Resistor_SMD:R_0805_2012Metric_Pad1.20x1.40mm_HandSolder, F.Cu at (92.8, 77.1)
- added R3: 510, Resistor_SMD:R_0805_2012Metric_Pad1.20x1.40mm_HandSolder, B.Cu at (134.6, 73.7)
- added R4: 510, Resistor_SMD:R_0805_2012Metric_Pad1.20x1.40mm_HandSolder, F.Cu at (95.0, 45.0)
- added R5: 510, Resistor_SMD:R_0805_2012Metric_Pad1.20x1.40mm_HandSolder, F.Cu at (96.2, 57.2)
- added R6: 510, Resistor_SMD:R_0805_2012Metric_Pad1.20x1.40mm_HandSolder, F.Cu at (94.7, 77.5)
- added R7: 510, Resistor_SMD:R_0805_2012Metric_Pad1.20x1.40mm_HandSolder, F.Cu at (101.6, 88.9)
- added R8: 510, Resistor_SMD:R_0805_2012Metric_Pad1.20x1.40mm_HandSolder, F.Cu at (94.0, 114.3)
- added R9: 510, Resistor_SMD:R_0805_2012Metric_Pad1.20x1.40mm_HandSolder, F.Cu at (94.0, 124.5)
- added S3: RDS-16S-1055-SMT, DigitalLogicFootprints:RDS16S1055SMT, F.Cu at (89.0, 104.0)
- added U2: SN74HC574DWR, DigitalLogicFootprints:SOIC127P1030X265-20N, B.Cu at (114.0, 50.8)
- U1: moved to B.Cu
- moved S2 38.5 mm to (90.5, 88.0), turned to 180 degrees
- moved S1 21.3 mm to (90.5, 72.0), turned to 180 degrees
- moved U1 17.2 mm to (111.5, 64.3)
Connections:
- S2 pad 3: CIRCUITBREAKRESET -> BUTTON
- U1 pad 1: unconnected-(U1-PD3-Pad1) -> ROTARYSWITCH3
- U1 pad 10: unconnected-(U1-PD6-Pad10) -> DIGIT1
- U1 pad 11: unconnected-(U1-PD7-Pad11) -> INPUT7
- U1 pad 12: unconnected-(U1-PB0-Pad12) -> DATA0
- U1 pad 13: unconnected-(U1-PB1-Pad13) -> DATA1
- U1 pad 14: unconnected-(U1-PB2-Pad14) -> DATA2
- U1 pad 15: unconnected-(U1-PB3-Pad15) -> DATA3
- U1 pad 16: unconnected-(U1-PB4-Pad16) -> DATA4
- U1 pad 17: unconnected-(U1-PB5-Pad17) -> DATA5
- U1 pad 19: unconnected-(U1-PE2-Pad19) -> CURRENTSENSE
- U1 pad 2: unconnected-(U1-PD4-Pad2) -> BUTTON
- U1 pad 22: unconnected-(U1-PE3-Pad22) -> RESET
- U1 pad 23: CURRENTSENSE -> INPUT0
- U1 pad 24: unconnected-(U1-PC1-Pad24) -> INPUT1
- U1 pad 25: unconnected-(U1-PC2-Pad25) -> INPUT2
- U1 pad 26: unconnected-(U1-PC3-Pad26) -> INPUT3
- U1 pad 27: CIRCUITBREAKRESET -> INPUT4
- U1 pad 28: MOSFET -> INPUT5
- U1 pad 29: RESET -> INPUT6
- U1 pad 3: unconnected-(U1-PE0-Pad3) -> MOSFET
- U1 pad 30: unconnected-(U1-PD0-Pad30) -> ROTARYSWITCH0
- U1 pad 31: unconnected-(U1-PD1-Pad31) -> ROTARYSWITCH1
- U1 pad 32: unconnected-(U1-PD2-Pad32) -> ROTARYSWITCH2
- U1 pad 6: unconnected-(U1-PE1-Pad6) -> DATACLK
- U1 pad 7: unconnected-(U1-XTAL1/PB6-Pad7) -> DATA6
- U1 pad 8: unconnected-(U1-XTAL2/PB7-Pad8) -> DATA7
- U1 pad 9: unconnected-(U1-PD5-Pad9) -> DIGIT0
Routing:
- net GND: track 436.6 -> 815.4 mm, vias 0 -> 11
- net +5V: track 0.00 -> 278.0 mm, vias 0 -> 2
- net INPUT0: track 0.00 -> 234.3 mm, vias 0 -> 4
- net INPUT7: track 0.00 -> 224.1 mm, vias 0 -> 2
- net VCC: track 456.8 -> 673.5 mm, vias 0 -> 11
- net INPUT6: track 0.00 -> 202.6 mm
- net INPUT1: track 0.00 -> 196.6 mm, vias 0 -> 5
- net DATA3: track 0.00 -> 183.1 mm, vias 0 -> 4
- net DATA5: track 0.00 -> 181.6 mm, vias 0 -> 3
- net DATA4: track 0.00 -> 180.8 mm, vias 0 -> 3
- net INPUT5: track 0.00 -> 169.9 mm, vias 0 -> 1
- net INPUT4: track 0.00 -> 168.3 mm, vias 0 -> 1
- net INPUT3: track 0.00 -> 157.0 mm, vias 0 -> 3
- net INPUT2: track 0.00 -> 149.8 mm, vias 0 -> 1
- net DATA6: track 0.00 -> 88.1 mm, vias 0 -> 2
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Other:
- board text added: "Board PCB Rev 1"
- board text added: "Jonathan Hess (jetsama.com)"
